File: KiCad/menorah555_main/menorah555.kicad_pcb (KiCad board)
At the start: 2 copper layers, 278.6 x 171.5 mm, 100 parts, among them J1 USB_B_Micro, J2 Jack5.5x2.1, J3 Plug5.5x2.1, Q1 MMBT3904, Q10 MJD31, Q2 MMBT3904, Q3 MMBT3904, Q4 MMBT3904, Q5 MMBT3904, Q6 MMBT3904, Q7 MMBT3904, Q8 MMBT3904, Q9 MMBT3904, SW1 SW_Reed, SW2 SW_Reed, SW3 SW_Reed, SW4 SW_Reed, SW5 SW_Reed, SW6 SW_Reed, SW7 SW_Reed, SW8 SW_Reed, SW9 SW_DPDT, U1 TLC555, U2 TLC555, U3 TLC555, U4 TLC555, U5 TLC555, U6 TLC555, U7 TLC555, U8 TLC555, U9 TLC555

Commit message: Updated design to KiCad 6.0.0
Initially the design was created in KiCad 5.1.12. To update it to KiCad
6.0.0 the path for the 3d models had to be changed from KISYS3DMOD to
KICAD6_3DMODEL_DIR. Additionally, the .wrl file were all changed to
.step files. No functional changes to the schematic or PCB were done
when updating to KiCad 6
Other:
- net class Default removed
- net class SHLD removed
