File: KiCad/menorah555_main/menorah555_main.kicad_pcb (KiCad board)
At the start: 2 copper layers, 278.6 x 166.1 mm, 93 parts, among them J1 USB_B_Micro, J2 Jack5.5x2.1, Q1 MMBT3904, Q10 MJD31, Q2 MMBT3904, Q3 MMBT3904, Q4 MMBT3904, Q5 MMBT3904, Q6 MMBT3904, Q7 MMBT3904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

Commit message: Fixed long turn-off time
Previously on the rev A PCB (PCB2002A), when power was turned off, the
shamash would take a very long time (> 20 minutes) to fully turn off.
Now a new diode, D11, has been added to drain the supercap when power is
turned off with the switch.
Parts:
- added D11: BAV99, Package_TO_SOT_SMD:SOT-23, F.Cu at (319.8, 154.1)
Routing:
- net Net-(D10-Pad2): track 126.7 -> 133.7 mm
- net Net-(D10-Pad1): track 9.82 -> 12.1 mm
Changed lines of the file:
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@@
   (net 66 "Net-(C17-Pad1)")
   (net 67 "Net-(C18-Pad1)")
+  (net 68 "unconnected-(D11-Pad1)")
   (footprint "Package_TO_SOT_SMD:SOT-23" (layer "F.Cu")
     (at 315.58 150.76 180)
@@
     )
   )
+  (footprint "Package_TO_SOT_SMD:SOT-23" (layer "F.Cu")
+    (at 319.75 154.1)
+    (descr "SOT, 3 Pin (https://www.jedec.org/system/files/docs/to-236h.pdf variant AB), generated with kicad-footprint-generator ipc_gullwing_generator.py")
+    (tags "SOT TO_SOT_SMD")
+    (property "Sheetfile" "menorah555_main.kicad_sch")
+    (property "Sheetname" "")
+    (property "Source" "Mouser 241-BAV99_R1_00001")
+    (attr smd)
+    (fp_text reference "D11" (at 3.4 0.15) (layer "F.SilkS")
+      (effects (font (size 1 1) (thickness 0.15)))
+    )
+    (fp_text value "BAV99" (at 0 2.4) (layer "F.Fab")
+      (effects (font (size 1 1) (thickness 0.15)))
+    )
+    (fp_text user "${REFERENCE}" (at 0 0) (layer "F.Fab")
+      (effects (font (size 0.32 0.32) (thickness 0.05)))
+    )
+    (fp_line (start 0 1.56) (end 0.65 1.56) (layer "F.SilkS") (width 0.12))
+    (fp_line (start 0 -1.56) (end -1.675 -1.56) (layer "F.SilkS") (width 0.12))
+    (fp_line (start 0 -1.56) (end 0.65 -1.56) (layer "F.SilkS") (width 0.12))
+    (fp_line (start 0 1.56) (end -0.65 1.56) (layer "F.SilkS") (width 0.12))
+    (fp_line (start 1.92 1.7) (end 1.92 -1.7) (layer "F.CrtYd") (width 0.05))
+    (fp_line (start 1.92 -1.7) (end -1.92 -1.7) (layer "F.CrtYd") (width 0.05))
+    (fp_line (start -1.92 -1.7) (end -1.92 1.7) (layer "F.CrtYd") (width 0.05))
+    (fp_line (start -1.92 1.7) (end 1.92 1.7) (layer "F.CrtYd") (width 0.05))
+    (fp_line (start 0.65 1.45) (end -0.65 1.45) (layer "F.Fab") (width 0.1))
+    (fp_line (start -0.325 -1.45) (end 0.65 -1.45) (layer "F.Fab") (width 0.1))
+    (fp_line (start 0.65 -1.45) (end 0.65 1.45) (layer "F.Fab") (width 0.1))
+    (fp_line (start -0.65 1.45) (end -0.65 -1.125) (layer "F.Fab") (width 0.1))
+    (fp_line (start -0.65 -1.125) (end -0.325 -1.45) (layer "F.Fab") (width 0.1))
+    (pad "1" smd roundrect locked (at -0.9375 -0.95) (size 1.475 0.6) (layers "F.Cu" "F.Paste" "F.Mask") (roundrect_rratio 0.25)
+      (net 68 "unconnected-(D11-Pad1)") (pinfunction "K") (pintype "passive+no_connect"))
+    (pad "2" smd roundrect locked (at -0.9375 0.95) (size 1.475 0.6) (layers "F.Cu" "F.Paste" "F.Mask") (roundrect_rratio 0.25)
+      (net 17 "Net-(D10-Pad1)") (pinfunction "A") (pintype "passive"))
+    (pad "3" smd roundrect locked (at 0.9375 0) (size 1.475 0.6) (layers "F.Cu" "F.Paste" "F.Mask") (roundrect_rratio 0.25)
+      (net 16 "Net-(D10-Pad2)") (pinfunction "K") (pintype "passive"))
+    (model "${KICAD6_3DMODEL_DIR}/Package_TO_SOT_SMD.3dshapes/SOT-23.wrl"
+      (offset (xyz 0 0 0))
+      (scale (xyz 1 1 1))
+      (rotate (xyz 0 0 0))
+    )
+  )
   (gr_line (start 78.2 121.6) (end 77.4 121.6) (layer "F.SilkS") (width 0.15))
   (gr_line (start 107.8 97.2) (end 107.8 98) (layer "F.SilkS") (width 0.15))
@@
   (segment (start 320.15 118.6) (end 318.75 120) (width 0.6) (layer "F.Cu") (net 1))
   (segment (start 230.15 100.2) (end 228.75 101.6) (width 0.6) (layer "F.Cu") (net 1))
-  (segment (start 205.2 138.4) (end 205.3 138.5) (width 0.25) (layer "F.Cu") (net 1))
   (via (at 170 83) (size 1) (drill 0.5) (layers "F.Cu" "B.Cu") (net 1))
   (via (at 174.4 115.4) (size 1) (drill 0.5) (layers "F.Cu" "B.Cu") (net 1))
@@
   (segment (start 258.295 97.075) (end 258.295 100.555) (width 0.6) (layer "F.Cu") (net 12))
   (segment (start 258.295 100.555) (end 258.25 100.6) (width 0.6) (layer "F.Cu") (net 12))
+  (segment (start 318.16 149.81) (end 320.6875 152.3375) (width 0.6) (layer "F.Cu") (net 16))
   (segment (start 315.2875 148.5175) (end 316.58 149.81) (width 0.6) (layer "F.Cu") (net 16))
+  (segment (start 320.6875 152.3375) (end 320.6875 154.1) (width 0.6) (layer "F.Cu") (net 16))
   (segment (start 309.69 148.5175) (end 310.0175 148.5175) (width 0.8) (layer "F.Cu") (net 16))
   (segment (start 309.69 148.5175) (end 302.8175 148.5175) (width 0.8) (layer "F.Cu") (net 16))
   (segment (start 302.8175 148.5175) (end 291.6 137.3) (width 0.8) (layer "F.Cu") (net 16))
   (segment (start 310.0175 148.5175) (end 315.2875 148.5175) (width 0.6) (layer "F.Cu") (net 16))
+  (segment (start 316.5175 149.81) (end 318.16 149.81) (width 0.6) (layer "F.Cu") (net 16))
   (segment (start 205.6 150.5) (end 200.5 150.5) (width 0.8) (layer "F.Cu") (net 16))
   (segment (start 291.6 137.3) (end 218.8 137.3) (width 0.8) (layer "F.Cu") (net 16))
@@
   (segment (start 314.26 156.16) (end 315.2925 156.16) (width 0.6) (layer "F.Cu") (net 17))
   (segment (start 316.58 154.8725) (end 315.2925 156.16) (width 0.6) (layer "F.Cu") (net 17))
+  (segment (start 316.7575 155.05) (end 316.58 154.8725) (width 0.6) (layer "F.Cu") (net 17))
   (segment (start 315.2925 156.16) (end 317.98 158.8475) (width 0.6) (layer "F.Cu") (net 17))
+  (segment (start 318.8125 155.05) (end 316.7575 155.05) (width 0.6) (layer "F.Cu") (net 17))
   (segment (start 78.45 143.8) (end 78.45 145.6375) (width 0.6) (layer "F.Cu") (net 22))
   (segment (start 78.45 145.6375) (end 78.4 145.6875) (width 0.6) (layer "F.Cu") (net 22))
@@
   (segment (start 286.52 139.9275) (end 289.8825 139.9275) (width 0.6) (layer "F.Cu") (net 28))
   (segment (start 289.8825 139.9275) (end 289.92 139.89) (width 0.6) (layer "F.Cu") (net 28))
-  (segment (start 309.69 156.15) (end 309.7 156.16) (width 0.6) (layer "F.Cu") (net 38))
-  (segment (start 309.7 153.1525) (end 309.69 153.1425) (width 0.8) (layer "F.Cu") (net 38))
   (segment (start 309.7 156.16) (end 309.7 153.1525) (width 0.8) (layer "F.Cu") (net 38))
   (segment (start 78.73 134) (end 78.73 137.3575) (width 0.6) (layer "F.Cu") (net 39))

Commit message: Made USB footprint hand-solderable
The USB footprint was changed to be an Amphenol 10118194-0001LF so that
it could be hand-soldered if desired.
Parts:
- J1: footprint 0_my_footprints:MOLEX_47590-0001 -> 0_my_footprints:AMPHENOL_10118194-0001LF
- moved J1 0.30 mm to (328.9, 205.2)
Routing:
- net +5V: track 897.6 -> 877.6 mm
- net GND: track 28.6 -> 36.7 mm
- net /RST_N: track 602.6 -> 601.3 mm
Other:
- outline, holes or cut-outs redrawn

Commit message: Eliminated silkscreen crossing edge cuts
The DRC was giving warnings for silkscreen that overlapped with edge
cuts because it was getting cut by the soldermask. The footprints for
the LEDs and the shamash power connector were updated to delete the
silkscreen outside of the board edge cuts
Parts:
- LED2, LED3, LED4, LED5, LED6, LED7, LED8, LED9: footprint 0_my_footprints:LED_D5.0mm_Horizontal_SMT_O3.81mm_Z3.0mm -> 0_menorah555:LED_D5.0mm_Horizontal_SMT_O3.81mm

Commit message: Offset the J2 model in Z direction
The 3d model for the J2 power jack has been offset by 2.35mm so that it
will make the main PCB and shamash PCB line up.
Parts:
- J2: footprint 0_my_footprints:Gravitech_CONSOCJ2155_2.1mm_5.5mm_Barrel_Jack -> 0_menorah555:Gravitech_CONSOCJ2155_2.1mm_5.5mm_Barrel_Jack_Z2.35
Changed lines of the file:
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@@
       (solder_mask_margin 0.5) (clearance 0.5))
   )
-  (footprint "0_my_footprints:Gravitech_CONSOCJ2155_2.1mm_5.5mm_Barrel_Jack" (layer "F.Cu")
+  (footprint "0_menorah555:Gravitech_CONSOCJ2155_2.1mm_5.5mm_Barrel_Jack_Z2.35" (layer "F.Cu")
     (at 200.5 150.5 -90)
     (descr "Gravitech CON-SOCJ-2155_1 2.1mm x 5.5mm Barrel Jack")
@@
     (property "Source" "Mouser 992-CON-SOCJ-2155 ")
     (attr through_hole)
-    (fp_text reference "J2" (at -6.7 -6 180) (layer "F.SilkS")
+    (fp_text reference "J2" (at -7.62 -6.35 -90) (layer "F.SilkS")
       (effects (font (size 1.27 1.27) (thickness 0.254)))
     )
-    (fp_text value "Jack5.5x2.1" (at -5.08 -1.27 90) (layer "F.Fab") hide
+    (fp_text value "Jack5.5x2.1" (at -5.08 -1.27 -90) (layer "F.Fab") hide
       (effects (font (size 1.27 1.27) (thickness 0.254)))
     )
-    (fp_text user "${REFERENCE}" (at -10.16 2.54 90) (layer "F.Fab")
+    (fp_text user "${REFERENCE}" (at -10.16 2.54 -90) (layer "F.Fab")
       (effects (font (size 1.27 1.27) (thickness 0.254)))
     )
+    (fp_line (start -13.6 4.5) (end -6.5 4.5) (layer "F.SilkS") (width 0.1))
     (fp_line (start 0 -4.5) (end -13.6 -4.5) (layer "F.SilkS") (width 0.1))
     (fp_line (start 0 -3) (end 0 -4.5) (layer "F.SilkS") (width 0.1))
-    (fp_line (start -13.6 4.5) (end -6.5 4.5) (layer "F.SilkS") (width 0.1))
     (fp_line (start -13.6 4.5) (end -13.6 -4.5) (layer "F.SilkS") (width 0.1))
     (fp_line (start 1.7 6.35) (end 1.7 -5) (layer "F.CrtYd") (width 0.1))
-    (fp_line (start -15.5 -5) (end -15.5 6.35) (layer "F.CrtYd") (width 0.1))
     (fp_line (start -15.5 6.35) (end 1.7 6.35) (layer "F.CrtYd") (width 0.1))
     (fp_line (start 1.7 -5) (end -15.5 -5) (layer "F.CrtYd") (width 0.1))
+    (fp_line (start -15.5 -5) (end -15.5 6.35) (layer "F.CrtYd") (width 0.1))
+    (fp_line (start 0 -4.5) (end -13.6 -4.5) (layer "F.Fab") (width 0.2))
+    (fp_line (start -13.6 -4.5) (end -13.6 4.5) (layer "F.Fab") (width 0.2))
     (fp_line (start 0 4.5) (end 0 -4.5) (layer "F.Fab") (width 0.2))
-    (fp_line (start 0 -4.5) (end -13.6 -4.5) (layer "F.Fab") (width 0.2))
     (fp_line (start -13.6 4.5) (end 0 4.5) (layer "F.Fab") (width 0.2))
-    (fp_line (start -13.6 -4.5) (end -13.6 4.5) (layer "F.Fab") (width 0.2))
-    (pad "1" thru_hole roundrect locked (at 0 0 270) (size 2.8 5) (drill oval 0.8 3) (layers *.Cu *.Mask) (roundrect_rratio 0.25)
+    (pad "1" thru_hole roundrect (at 0 0 270) (size 2.8 5) (drill oval 0.8 3) (layers *.Cu *.Mask) (roundrect_rratio 0.25)
       (net 16 "Net-(D10-Pad2)") (pintype "passive"))
-    (pad "2" thru_hole roundrect locked (at -6 0 270) (size 2.8 5) (drill oval 0.8 3) (layers *.Cu *.Mask) (roundrect_rratio 0.25)
+    (pad "2" thru_hole roundrect (at -6 0 270) (size 2.8 5) (drill oval 0.8 3) (layers *.Cu *.Mask) (roundrect_rratio 0.25)
       (net 1 "GND") (pintype "passive"))
-    (pad "3" thru_hole roundrect locked (at -3 4.6 270) (size 5 2.8) (drill oval 3 0.8) (layers *.Cu *.Mask) (roundrect_rratio 0.25)
+    (pad "3" thru_hole roundrect (at -3 4.6 270) (size 5 2.8) (drill oval 3 0.8) (layers *.Cu *.Mask) (roundrect_rratio 0.25)
       (net 20 "unconnected-(J2-Pad3)") (pintype "passive+no_connect"))
-    (model "${MY3DMODELS}/CON-SOCJ-2155.stp"
-      (offset (xyz 0 0 0))
+    (model "${KIPRJMOD}/project_libraries/project_3dmodels/CON-SOCJ-2155.stp"
+      (offset (xyz 0 0 2.35))
       (scale (xyz 1 1 1))
       (rotate (xyz 0 0 0))

Commit message: Updated slide switch to ground the case
The Nidec slide switch case had pins named 'M' that were not on the
schematic, so they did not get connected on the PCB. Now those pins have
been added to the symbol and connected to ground.
Connections:
- SW9 pad M: (no net) -> GND
Changed lines of the file:
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@@
     (pad "6" thru_hole oval locked (at 4 1.25 270) (size 2.5 1.5) (drill oval 1.4 0.8) (layers *.Cu *.Mask)
       (net 1 "GND") (pinfunction "C") (pintype "passive"))
-    (pad "M" thru_hole oval locked (at 8.25 0 270) (size 2.8 4) (drill oval 1.4 2.3) (layers *.Cu *.Mask))
-    (pad "M" thru_hole oval locked (at -8.25 0 270) (size 2.8 4) (drill oval 1.4 2.3) (layers *.Cu *.Mask))
+    (pad "M" thru_hole oval locked (at 8.25 0 270) (size 2.8 4) (drill oval 1.4 2.3) (layers *.Cu *.Mask)
+      (net 1 "GND") (pinfunction "M") (pintype "passive"))
+    (pad "M" thru_hole oval locked (at -8.25 0 270) (size 2.8 4) (drill oval 1.4 2.3) (layers *.Cu *.Mask)
+      (net 1 "GND") (pinfunction "M") (pintype "passive"))
     (model "${KICAD6_3DMODEL_DIR}/Button_Switch_THT.3dshapes/SW_CuK_JS202011CQN_DPDT_Straight.step"
       (offset (xyz -4.5 3.5 0))

Commit message: Added silkscreen 2mm stripe at edge
For aesthetic reasons, a 2mm silkscreen strip was added around the board
on top and bottom. Gerbers were also generated
Parts:
- C10, C11, C12, C13, C14, C15, C16, C9: footprint 0_my_footprints:CP_Radial_Horizontal_D8.0mm_L12.0mm_P3.50mm -> 0_menorah555:CP_Radial_Horizontal_D8.0mm_L12.0mm_P3.50mm_narrow
- SW1, SW2, SW3, SW4, SW5, SW6, SW7, SW8: footprint 0_my_footprints:SW_SPST_REED_59170-1-S-00-D -> 0_menorah555:SW_SPST_REED_59170-1-S-00-D_1side
- moved LOGO2 7.98 mm to (318.8, 204.9)
Other:
- outline, holes or cut-outs redrawn
