File: KiCad/menorah555_shamash/menorah555_shamash.kicad_sch (KiCad schematic)
At the start: 8 parts, among them J3 Plug5.5x2.1

Commit message: Eliminated silkscreen crossing edge cuts
The DRC was giving warnings for silkscreen that overlapped with edge
cuts because it was getting cut by the soldermask. The footprints for
the LEDs and the shamash power connector were updated to delete the
silkscreen outside of the board edge cuts
Parts:
- LED1: footprint 0_my_footprints:LED_D5.0mm_Horizontal_SMT_O3.81mm_Z3.0mm -> 0_project_footprints:LED_D5.0mm_Horizontal_SMT_O3.81mm
Changed lines of the file:
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@@
       (effects (font (size 1.27 1.27)) (justify right))
     )
-    (property "Footprint" "0_my_footprints:LED_D5.0mm_Horizontal_SMT_O3.81mm_Z3.0mm" (id 2) (at 113.03 64.77 0)
+    (property "Footprint" "0_project_footprints:LED_D5.0mm_Horizontal_SMT_O3.81mm" (id 2) (at 113.03 64.77 0)
       (effects (font (size 1.27 1.27)) hide)
     )
@@
     )
     (path "/00000000-0000-0000-0000-000061bf0f3d"
-      (reference "LED1") (unit 1) (value "Y FLCKR LED") (footprint "0_my_footprints:LED_D5.0mm_Horizontal_SMT_O3.81mm_Z3.0mm")
+      (reference "LED1") (unit 1) (value "Y FLCKR LED") (footprint "0_project_footprints:LED_D5.0mm_Horizontal_SMT_O3.81mm")
     )
     (path "/00000000-0000-0000-0000-000060735e73"
